File: hardware/color-spray.kicad_pcb (KiCad board)
At the start: 2 copper layers, 76.2 x 68.6 mm, 38 parts, among them J1 MIDI Input, J2 ARGB_XLR3, J3 ARGB, J4 DMX_XLR3, J5 External RGBW Power, J6 RGBW, Q1 IRLB8721PBF, Q2 IRLB8721PBF, Q3 IRLB8721PBF, Q4 IRLB8721PBF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

Commit message: Reorganization and renaming.
Other:
- board text added: "dcdalrymple.com/color-spray"
- board text removed: "dcdalrymple.com/arduino-midi-argb-dmx"

Commit message: Added OSHWA certification mark to PCB and README.
Parts:
- removed the REF** at (141.0, 123.2)
- added G***: LOGO, oshw-mark:oshw-mark_10mm, B.Cu at (141.0, 123.2)
Other:
- board text added: "Color Spray"
